Commit message: Fixed description file

File: reach_description/description/bravo_7/end_effectors/standard_jaws.urdf.xacro (robot description, xacro)
@@ -9,5 +9,5 @@
       <visual>
         <geometry>
-          <mesh filename="$(find reach_description)/meshes/bravo_7/end_effectors/RS2-257.stl" />
+          <mesh filename="file://$(find reach_description)/meshes/bravo_7/end_effectors/RS2-257.stl" />
         </geometry>
         <material name="${prefix}black" />
@@ -27,8 +27,8 @@
         <geometry>
           <cylinder length="0.02"
-                    radius="0.05" />
+                    radius="0.04" />
         </geometry>
-        <origin xyz="0.01 0 0.00"
-                rpy="0 1.5707 0" />
+        <origin xyz="0.0 0.0 0.13074999999999998"
+                rpy="0.0 0.0 0.0" />
       </collision>
     </link>
@@ -36,5 +36,5 @@
       <visual>
         <geometry>
-          <mesh filename="$(find reach_description)/meshes/bravo_7/end_effectors/RS2-300.stl" />
+          <mesh filename="file://$(find reach_description)/meshes/bravo_7/end_effectors/RS2-300.stl" />
         </geometry>
         <material name="${prefix}black" />
@@ -42,5 +42,5 @@
       <inertial>
         <mass value="0.24" />
-        <origin xyz="0.05 0.0 0" />
+        <origin xyz="0.05 0.0 0.0" />
         <inertia ixx="${244 * 1e-6}"
                  ixy="${-12 * 1e-6}"
@@ -52,5 +52,5 @@
       <collision>
         <geometry>
-          <mesh filename="$(find reach_description)/meshes/bravo_7/end_effectors/RS2-300.stl" />
+          <mesh filename="file://$(find reach_description)/meshes/bravo_7/end_effectors/RS2-300.stl" />
         </geometry>
       </collision>
@@ -59,5 +59,5 @@
       <visual>
         <geometry>
-          <mesh filename="$(find reach_description)/meshes/bravo_7/end_effectors/RS2-301.stl" />
+          <mesh filename="file://$(find reach_description)/meshes/bravo_7/end_effectors/RS2-301.stl" />
         </geometry>
         <material name="${prefix}black" />
@@ -65,5 +65,5 @@
       <inertial>
         <mass value="0.24" />
-        <origin xyz="0.05 0.0 0" />
+        <origin xyz="0.05 0.0 0.0" />
         <inertia ixx="${244 * 1e-6}"
                  ixy="${-12 * 1e-6}"
@@ -75,5 +75,5 @@
       <collision>
         <geometry>
-          <mesh filename="$(find reach_description)/meshes/bravo_7/end_effectors/RS2-301.stl" />
+          <mesh filename="file://$(find reach_description)/meshes/bravo_7/end_effectors/RS2-301.stl" />
         </geometry>
       </collision>
@@ -84,15 +84,15 @@
       <parent link="${parent}" />
       <child link="${prefix}base_link" />
-      <origin xyz="0 0 0"
-              rpy="0 0 0" />
+      <origin xyz="0.0 0.0 0.0"
+              rpy="0.0 0.0 0.0" />
     </joint>
     <joint name="${prefix}rs2_300_joint"
            type="revolute">
-      <origin xyz="0.0097 -0.033 0"
-              rpy="0 0 0" />
+      <origin xyz="2.3214757534187783e-06 0.0268 0.15484999988818982"
+              rpy="0.0 -1.5706999999997038 0.0" />
       <parent link="${prefix}base_link" />
       <child link="${prefix}rs2_300_link" />
       <axis xyz="0 0 -1" />
-      <limit lower="0"
+      <limit lower="0.0"
              upper="1.0"
              effort="400"
@@ -104,6 +104,6 @@
     <joint name="${prefix}rs2_301_joint"
            type="revolute">
-      <origin xyz="0.0097 0.033 0"
-              rpy="0 0 0" />
+      <origin xyz="2.3214757534187783e-06 -0.0268 0.15484999988818982"
+              rpy="0.0 -1.5706999999997038 0.0" />
       <parent link="${prefix}base_link" />
       <child link="${prefix}rs2_301_link" />

File: reach_description/description/bravo_7/urdf.xacro (robot description, xacro)
@@ -21,5 +21,5 @@
         <material name="${prefix}black" />
         <geometry>
-          <mesh filename="$(find reach_description)/meshes/bravo_7/1019-A.stl" />
+          <mesh filename="file://$(find reach_description)/meshes/bravo_7/1019-A.stl" />
         </geometry>
       </visual>
@@ -61,5 +61,5 @@
       <visual>
         <geometry>
-          <mesh filename="$(find reach_description)/meshes/bravo_7/1013-A.stl" />
+          <mesh filename="file://$(find reach_description)/meshes/bravo_7/1013-A.stl" />
         </geometry>
         <material name="${prefix}black" />
@@ -69,5 +69,5 @@
       <visual>
         <geometry>
-          <mesh filename="$(find reach_description)/meshes/bravo_7/1019-B.stl" />
+          <mesh filename="file://$(find reach_description)/meshes/bravo_7/1019-B.stl" />
         </geometry>
         <material name="${prefix}black" />
@@ -106,5 +106,5 @@
       <visual>
         <geometry>
-          <mesh filename="$(find reach_description)/meshes/bravo_7/1013-B.stl" />
+          <mesh filename="file://$(find reach_description)/meshes/bravo_7/1013-B.stl" />
         </geometry>
         <material name="${prefix}black" />
@@ -114,5 +114,5 @@
       <visual>
         <geometry>
-          <mesh filename="$(find reach_description)/meshes/bravo_7/RS2-1026-A.stl" />
+          <mesh filename="file://$(find reach_description)/meshes/bravo_7/RS2-1026-A.stl" />
         </geometry>
         <material name="${prefix}black" />
@@ -122,5 +122,5 @@
       <visual>
         <geometry>
-          <mesh filename="$(find reach_description)/meshes/bravo_7/1030.stl" />
+          <mesh filename="file://$(find reach_description)/meshes/bravo_7/1030.stl" />
         </geometry>
         <material name="${prefix}black" />
@@ -223,5 +223,5 @@
       <visual>
         <geometry>
-          <mesh filename="$(find reach_description)/meshes/bravo_7/RS2-1026-B.stl" />
+          <mesh filename="file://$(find reach_description)/meshes/bravo_7/RS2-1026-B.stl" />
         </geometry>
         <material name="${prefix}black" />
@@ -260,5 +260,5 @@
       <visual>
         <geometry>
-          <mesh filename="$(find reach_description)/meshes/bravo_7/RS2-1026-C.stl" />
+          <mesh filename="file://$(find reach_description)/meshes/bravo_7/RS2-1026-C.stl" />
         </geometry>
         <material name="${prefix}black" />
@@ -268,5 +268,5 @@
       <visual>
         <geometry>
-          <mesh filename="$(find reach_description)/meshes/bravo_7/RS2-1023-A.stl" />
+          <mesh filename="file://$(find reach_description)/meshes/bravo_7/RS2-1023-A.stl" />
         </geometry>
         <material name="${prefix}black" />
@@ -313,5 +313,5 @@
       <visual>
         <geometry>
-          <mesh filename="$(find reach_description)/meshes/bravo_7/RS2-1023-B.stl" />
+          <mesh filename="file://$(find reach_description)/meshes/bravo_7/RS2-1023-B.stl" />
         </geometry>
         <material name="${prefix}black" />
@@ -371,5 +371,5 @@
         <visual>
           <geometry>
-            <mesh filename="$(find reach_description)/meshes/bravo_7/RS2-1023-C.stl" />
+            <mesh filename="file://$(find reach_description)/meshes/bravo_7/RS2-1023-C.stl" />
           </geometry>
           <material name="${prefix}black" />
@@ -379,5 +379,5 @@
         <visual>
           <geometry>
-            <mesh filename="$(find reach_description)/meshes/bravo_7/1038.stl" />
+            <mesh filename="file://$(find reach_description)/meshes/bravo_7/1038.stl" />
           </geometry>
           <material name="${prefix}black" />
@@ -413,5 +413,4 @@
         </collision>
       </link>
-      <insert_block name="end_effector" />
     </xacro:if>
     <xacro:unless value="${use_ft_sensor}">
@@ -430,5 +429,5 @@
         <visual>
           <geometry>
-            <mesh filename="$(find reach_description)/meshes/bravo_7/RS2-1023-C.stl" />
+            <mesh filename="file://$(find reach_description)/meshes/bravo_7/RS2-1023-C.stl" />
           </geometry>
           <material name="${prefix}black" />
@@ -438,5 +437,5 @@
         <visual>
           <geometry>
-            <mesh filename="$(find reach_description)/meshes/bravo_7/1038.stl" />
+            <mesh filename="file://$(find reach_description)/meshes/bravo_7/1038.stl" />
           </geometry>
           <material name="${prefix}black" />
@@ -475,11 +474,4 @@
       </inertial>
     </link>
-    <xacro:include filename="$(find reach_description)/description/bravo_7/end_effectors/standard_jaws.urdf.xacro" />
-    <xacro:standard_jaws_urdf parent="${prefix}ee_base_link"
-                              prefix="${prefix}standard_jaws_"
-                              axis_a="${prefix}axis_a">
-      <origin xyz="0 0 0"
-              rpy="0 0 0" />
-    </xacro:standard_jaws_urdf>
     <!-- Joints -->
     <joint name="${prefix}base_joint"
@@ -615,4 +607,11 @@
              upper="0.035" />
     </joint>
+    <xacro:include filename="$(find reach_description)/description/bravo_7/end_effectors/standard_jaws.urdf.xacro" />
+    <xacro:standard_jaws_urdf parent="${prefix}1023_1_joint_link"
+                              prefix="${prefix}standard_jaws_"
+                              axis_a="${prefix}axis_a">
+      <origin xyz="0 0 0"
+              rpy="0 0 0" />
+    </xacro:standard_jaws_urdf>
   </xacro:macro>
 </robot>

Commit message: Finished initial impedance controller and cleaned up urdf

File: reach_description/description/bravo_7/end_effectors/standard_jaws.urdf.xacro (robot description, xacro)
@@ -12,15 +12,17 @@
         </geometry>
         <material name="${prefix}black" />
-        <origin xyz="0.0 0.0 0.13074999999999998"
-                rpy="0.0 -1.5706999999997038 0.0" />
+        <origin xyz="0.0 0.0 0.13075"
+                rpy="0.0 -1.5707 0.0" />
       </visual>
       <inertial>
-        <mass value="0.01" />
-        <inertia ixx="0.0001"
+        <origin xyz="0.008269 0.0 0.13075"
+                rpy="0.0 -0.0 0.0" />
+        <mass value="0.64" />
+        <inertia ixx="0.0003"
                  ixy="0.0"
                  ixz="0.0"
-                 iyy="0.0001"
+                 iyy="0.002202"
                  iyz="0.0"
-                 izz="0.0001" />
+                 izz="0.002181" />
       </inertial>
       <collision>
@@ -29,5 +31,5 @@
                     radius="0.04" />
         </geometry>
-        <origin xyz="0.0 0.0 0.13074999999999998"
+        <origin xyz="0.0 0.0 0.13075"
                 rpy="0.0 0.0 0.0" />
       </collision>
@@ -43,10 +45,10 @@
         <mass value="0.24" />
         <origin xyz="0.05 0.0 0.0" />
-        <inertia ixx="${244 * 1e-6}"
-                 ixy="${-12 * 1e-6}"
-                 ixz="${0 * 1e-6}"
-                 iyy="${1130 * 1e-6}"
-                 iyz="${1 * 1e-6}"
-                 izz="${1178 * 1e-6}" />
+        <inertia ixx="0.001"
+                 ixy="0.0"
+                 ixz="0.0"
+                 iyy="0.001"
+                 iyz="0.0"
+                 izz="0.001" />
       </inertial>
       <collision>
@@ -66,10 +68,10 @@
         <mass value="0.24" />
         <origin xyz="0.05 0.0 0.0" />
-        <inertia ixx="${244 * 1e-6}"
-                 ixy="${-12 * 1e-6}"
-                 ixz="${0 * 1e-6}"
-                 iyy="${1130 * 1e-6}"
-                 iyz="${1 * 1e-6}"
-                 izz="${1178 * 1e-6}" />
+        <inertia ixx="0.001"
+                 ixy="0.0"
+                 ixz="0.0"
+                 iyy="0.001"
+                 iyz="0.0"
+                 izz="0.001" />
       </inertial>
       <collision>

File: reach_description/description/bravo_7/urdf.xacro (robot description, xacro)
@@ -26,12 +26,12 @@
       <inertial>
         <origin xyz="0.052500000000000005 -0.0010000053071760658 0.033650002653596835"
-                rpy="0.0 -0.0 0.0" />
+                rpy="0.0 0.0 0.0" />
         <mass value="1.85" />
-        <inertia ixx="0.0001767933750000004"
-                 ixy="-0.010800269063967364"
-                 ixz="-0.010757269071928286"
-                 iyy="-0.008187269162146547"
-                 iyz="-0.01078726772655808"
-                 izz="-0.005309062462853453" />
+        <inertia ixx="0.00018"
+                 ixy="-0.01080"
+                 ixz="-0.01076"
+                 iyy="-0.00819"
+                 iyz="-0.01079"
+                 izz="-0.00531" />
       </inertial>
       <collision>
@@ -76,13 +76,13 @@
       </visual>
       <inertial>
-        <origin xyz="0.029000053072066954 -0.010000103489825904 0.05364997346396829"
-                rpy="0.0 -0.0 0.0" />
+        <origin xyz="0.0290000 -0.010000 0.053650"
+                rpy="0.0 0.0 0.0" />
         <mass value="1.62" />
-        <inertia ixx="-7.4169231311085534e-06"
-                 ixy="-0.0029550371991257053"
-                 ixz="-0.004212035657385413"
-                 iyy="0.0010209661974629213"
-                 iyz="-0.002844035049716061"
-                 izz="0.002385381825668186" />
+        <inertia ixx="0.0"
+                 ixy="-0.00296"
+                 ixz="-0.00421"
+                 iyy="0.00102"
+                 iyz="-0.00284"
+                 izz="0.00239" />
       </inertial>
       <collision>
@@ -117,5 +117,5 @@
         </geometry>
         <material name="${prefix}black" />
-        <origin xyz="0.04600000000128156 4.829533423884964e-07 -0.23533999999935923"
+        <origin xyz="0.046 0.0 -0.23534"
                 rpy="3.14159 -0.0 3.14159" />
       </visual>
@@ -129,13 +129,13 @@
       </visual>
       <inertial>
-        <origin xyz="0.02614393591762409 -0.004000726999431309 -0.17620840523390582"
+        <origin xyz="0.02614 -0.004 -0.17621"
                 rpy="0.0 -0.0 0.0" />
         <mass value="2.12" />
-        <inertia ixx="0.03522180708867557"
-                 ixy="-2.5616015376588342e-05"
-                 ixz="-0.0013021484721849014"
-                 iyy="0.03597802003044357"
-                 iyz="-0.0031539607831752277"
-                 izz="0.003361250024861972" />
+        <inertia ixx="0.03522"
+                 ixy="-0.00002"
+                 ixz="-0.00130"
+                 iyy="0.03598"
+                 iyz="-0.00315"
+                 izz="0.00336" />
       </inertial>
       <collision>
@@ -160,5 +160,5 @@
                     length="0.059" />
         </geometry>
-        <origin xyz="0.04600000000148929 5.612342412921263e-07 -0.26483999999925534"
+        <origin xyz="0.046 0.0 -0.26484"
                 rpy="3.14159 -0.0 3.14159" />
       </collision>
@@ -168,6 +168,6 @@
                     length="0.0599" />
         </geometry>
-        <origin xyz="0.005199961922827123 -0.014349252218295189 -0.294340038078165"
-                rpy="-1.5708953071795866 -0.0 3.14159" />
+        <origin xyz="0.005290 -0.01435 -0.29434"
+                rpy="-1.5707 -0.0 3.14159" />
       </collision>
       <collision>
@@ -176,5 +176,5 @@
                     length="0.03033333" />
         </geometry>
-        <origin xyz="0.046000000000106796 4.0246094175109416e-08 -0.0685066599999466"
+        <origin xyz="0.046 0.0 -0.06851"
                 rpy="3.14159 -0.0 3.14159" />
       </collision>
@@ -184,5 +184,5 @@
                     length="0.03033333" />
         </geometry>
-        <origin xyz="0.04600000000032039 1.207383355971241e-07 -0.0988399999998398"
+        <origin xyz="0.046 0.0 -0.09884"
                 rpy="3.14159 -0.0 3.14159" />
       </collision>
@@ -192,5 +192,5 @@
                     length="0.03033333" />
         </geometry>
-        <origin xyz="0.04600000000053398 2.0123055844401027e-07 -0.129173332999733"
+        <origin xyz="0.046 0.0 -0.12917"
                 rpy="3.14159 -0.0 3.14159" />
       </collision>
@@ -200,5 +200,5 @@
                     length="0.03033333" />
         </geometry>
-        <origin xyz="0.046000000000747575 2.817227828830503e-07 -0.1595066665996262"
+        <origin xyz="0.046 0.0 -0.15951"
                 rpy="3.14159 -0.0 3.14159" />
       </collision>
@@ -208,5 +208,5 @@
                     length="0.03033333" />
         </geometry>
-        <origin xyz="0.04600000000096117 3.6221500679137236e-07 -0.18983999999951942"
+        <origin xyz="0.046 0.0 -0.18984"
                 rpy="3.14159 -0.0 3.14159" />
       </collision>
@@ -216,5 +216,5 @@
                     length="0.03033333" />
         </geometry>
-        <origin xyz="0.04600000000117476 4.427071420697953e-07 -0.22017329999941262"
+        <origin xyz="0.046 0.0 -0.22017"
                 rpy="3.14159 -0.0 3.14159" />
       </collision>
@@ -230,13 +230,13 @@
       </visual>
       <inertial>
-        <origin xyz="0.031063964725062076 0.002998228717415121 -0.04499613595612657"
+        <origin xyz="0.03106 0.003 -0.045"
                 rpy="0.0 -0.0 0.0" />
         <mass value="1.33" />
-        <inertia ixx="0.0018075916378076167"
-                 ixy="0.00014318762193144414"
-                 ixz="0.0003851922094691543"
-                 iyy="0.0020111672541860653"
-                 iyz="-0.0002098175940630606"
-                 izz="0.001545577033243905" />
+        <inertia ixx="0.00181"
+                 ixy="0.00014"
+                 ixz="0.00039"
+                 iyy="0.00201"
+                 iyz="-0.00021"
+                 izz="0.00155" />
       </inertial>
       <collision>
@@ -245,5 +245,5 @@
                     length="0.02335" />
         </geometry>
-        <origin xyz="0.0 0.027275 0.0"
+        <origin xyz="0.0 0.02728 0.0"
                 rpy="1.5707 0.0 0.0" />
       </collision>
@@ -275,13 +275,13 @@
       </visual>
       <inertial>
-        <origin xyz="-0.030926349610074382 0.012001163718658751 0.056948306126308565"
+        <origin xyz="-0.03093 0.012 0.05695"
                 rpy="0.0 -0.0 0.0" />
         <mass value="1.33" />
-        <inertia ixx="-0.00832916419325029"
-                 ixy="-0.010143824151758763"
-                 ixz="-0.009682830984713842"
-                 iyy="-0.007647783076280421"
-                 iyz="-0.0105877952718513"
-                 izz="0.001514369533161315" />
+        <inertia ixx="-0.00833"
+                 ixy="-0.01014"
+                 ixz="-0.00968"
+                 iyy="-0.00765"
+                 iyz="-0.01059"
+                 izz="0.00151" />
       </inertial>
       <collision>
@@ -306,5 +306,5 @@
                     length="0.0599" />
         </geometry>
-        <origin xyz="-0.04079996192084282 0.014350108266413046 0.0644"
+        <origin xyz="-0.0408 0.01435 0.0644"
                 rpy="1.5707 -0.0 3.14159" />
       </collision>
@@ -320,13 +320,13 @@
       </visual>
       <inertial>
-        <origin xyz="0.03882206784524773 -0.006000269377738013 -0.041913219531621276"
+        <origin xyz="0.03882 -0.006 -0.04191"
                 rpy="0.0 -0.0 0.0" />
         <mass value="0.97" />
-        <inertia ixx="0.0012635074957551597"
-                 ixy="4.859518648201744e-05"
-                 ixz="0.00027856597958993856"
-                 iyy="0.0014435491024125883"
-                 iyz="-0.00025641638880114734"
-                 izz="0.0011460308711732192" />
+        <inertia ixx="0.00126"
+                 ixy="0.00004"
+                 ixz="0.00028"
+                 iyy="0.00144"
+                 iyz="-0.00026"
+                 izz="0.00115" />
       </inertial>
       <collision>
@@ -386,13 +386,13 @@
         </visual>
         <inertial>
-          <origin xyz="-0.007856122583731653 1.191782894075085e-06 0.06886021849973584"
+          <origin xyz="-0.007856122583731653 0.0 0.06886021849973584"
                   rpy="0.0 -0.0 0.0" />
           <mass value="1.35" />
-          <inertia ixx="-0.0070153399422235915"
-                   ixy="-0.009640678120463793"
-                   ixz="-0.009618302820342164"
-                   iyy="-0.006090679776636699"
-                   iyz="-0.00963571107587032"
-                   izz="0.0011986599361994638" />
+          <inertia ixx="-0.00702"
+                   ixy="-0.00964"
+                   ixz="-0.00962"
+                   iyy="-0.00609"
+                   iyz="-0.00964"
+                   izz="0.00120" />
         </inertial>
         <collision>
@@ -417,13 +417,13 @@
       <link name="${prefix}1023_1_joint_link">
         <inertial>
-          <origin xyz="-0.007848348345388155 8.383467019698216e-07 0.04286021966442238"
+          <origin xyz="-0.00785 0.0 0.04286"
                   rpy="0.0 -0.0 0.0" />
           <mass value="1.09" />
-          <inertia ixx="-0.005739665883907044"
-                   ixy="-0.007783149016640456"
-                   ixz="-0.007767867282695909"
-                   iyy="-0.005797148921426273"
-                   iyz="-0.007782161916684913"
-                   izz="0.0009685169067404991" />
+          <inertia ixx="-0.00574"
+                   ixy="-0.00778"
+                   ixz="-0.00777"
+                   iyy="-0.00579"
+                   iyz="-0.00778"
+                   izz="0.000969" />
         </inertial>
         <visual>
@@ -462,14 +462,21 @@
     </xacro:unless>
     <link name="${prefix}push_rod">
+      <visual>
+        <geometry>
+          <cylinder length="0.01"
+                    radius="0.0001" />
+        </geometry>
+        <material name="${prefix}black" />
+        <origin xyz="0.0 0.0 0.0"
+                rpy="0.0 -0.0 0.0" />
+      </visual>
       <inertial>
-        <origin xyz="0.008269061206615146 2.1481704501120766e-06 -0.00012210240446196524"
-                rpy="0.0 -0.0 0.0" />
-        <mass value="0.64" />
-        <inertia ixx="0.0003082092929784328"
-                 ixy="-5.6822416478701867e-05"
-                 ixz="-7.455807417347965e-05"
-                 iyy="0.0022022041006320905"
-                 iyz="-5.579658104299784e-05"
-                 izz="0.0021819948567845843" />
+        <mass value="0.01" />
+        <inertia ixx="0.0001"
+                 ixy="0.0"
+                 ixz="0.0"
+                 iyy="0.0001"
+                 iyz="0.0"
+                 izz="0.0001" />
       </inertial>
     </link>
@@ -516,5 +523,5 @@
       <child link="${prefix}1026_0_joint_link" />
       <axis xyz=" 0 -1 0" />
-      <origin xyz="0.005200000001840656 7.477816037645476e-07 -0.2943399999991515"
+      <origin xyz="0.0052 0.0 -0.29434"
               rpy="3.14159 -0.0 3.14159" />
       <dynamics damping="${joint_damping}"
@@ -544,5 +551,5 @@
       <child link="${prefix}1023_0_joint_link" />
       <axis xyz=" 0 -1 0" />
-      <origin xyz="-0.040799999999856354 1.082664635687914e-07 0.0644"
+      <origin xyz="-0.0408 0.0 0.0644"
               rpy="0.0 -0.0 3.14159" />
       <dynamics damping="${joint_damping}"
@@ -598,6 +605,6 @@
       <child link="${prefix}push_rod" />
       <axis xyz="0 0 1" />
-      <origin xyz="-0.008999999958245167 0.0 0.1307508669411527"
-              rpy="0.0 -1.5706999999997038 0.0" />
+      <origin xyz="-0.009 0.0 0.13075"
+              rpy="0.0 -1.5707 0.0" />
       <dynamics damping="${prismatic_joint_damping}"
                 friction="${joint_friction}" />
