Commit message: Cleaned up package structure and split tcp/robot controllers

File: reach_description/description/alpha_5/standard_jaws/alpha_5.config.xacro (robot description, xacro)
@@ -1,9 +1,9 @@
 <?xml version="1.0"?>
-<robot name="alpha"
+<robot name="alpha_5"
        xmlns:xacro="http://ros.org/wiki/xacro">
   <!-- import main macros -->
   <xacro:include filename="$(find reach_description)/description/alpha_5/urdf.xacro" />
   <xacro:include filename="$(find reach_description)/description/alpha_5/ros2_control.xacro" />
-  <xacro:include filename="$(find reach_description)/description/alpha_5/end_effectors/standard_jaws.urdf.xacro" />
+  <xacro:include filename="$(find reach_description)/description/alpha_5/standard_jaws/standard_jaws.urdf.xacro" />
   <xacro:include filename="$(find reach_description)/description/alpha_5/gz.xacro" />
   <!-- parameters -->
@@ -38,5 +38,5 @@
   <xacro:standard_jaws parent="${prefix}rs1_124_link"
                        prefix="${prefix}"
-                       axis_a="${prefix}axis_a">
+                       mimic_joint="${prefix}axis_a">
   </xacro:standard_jaws>
   <!-- ros2_control interface -->
@@ -46,4 +46,5 @@
                         use_sim="${use_sim}"
                         use_mock_hardware="$(arg use_mock_hardware)" />
+  <!-- gazebo configuration -->
   <xacro:if value="$(arg use_sim)">
     <xacro:alpha_5_gazebo prefix="${prefix}"

File: reach_description/description/alpha_5/standard_jaws/standard_jaws.urdf.xacro (robot description, xacro)
@@ -2,5 +2,6 @@
 <robot xmlns:xacro="http://ros.org/wiki/xacro">
   <xacro:macro name="standard_jaws"
-               params="parent prefix axis_a">
+               params="parent prefix mimic_joint">
+    <!-- links -->
     <link name="${prefix}rs1_130_link">
       <visual>
@@ -57,4 +58,5 @@
       </inertial>
     </link>
+    <!-- define a tcp link for planning/control purposes -->
     <link name="${prefix}tcp">
       <inertial>
@@ -68,4 +70,5 @@
       </inertial>
     </link>
+    <!-- joints -->
     <joint name="${prefix}rs1_130_joint"
            type="revolute">
@@ -79,5 +82,5 @@
              effort="10"
              velocity="10" />
-      <mimic joint="${axis_a}"
+      <mimic joint="${mimic_joint}"
              multiplier="51"
              offset="0" />

Commit message: Enable mount rotation configuration

File: reach_description/description/alpha_5/standard_jaws/alpha_5.config.xacro (robot description, xacro)
@@ -20,4 +20,6 @@
   <xacro:arg name="controllers_file"
              default="$(find reach_description)/config/alpha_5/controllers.yaml" />
+  <xacro:arg name="mount_rotation"
+             default="0" />
   <!-- initial positions used for simulation -->
   <xacro:arg name="initial_positions_file"
@@ -32,6 +34,6 @@
   <xacro:alpha_5_urdf parent="$(arg parent)"
                       prefix="${prefix}">
-    <origin xyz="0 0 0"
-            rpy="0 0 0" />
+    <origin xyz="0.0374 0 0.0225"
+            rpy="$(arg mount_rotation) 0 0" />
   </xacro:alpha_5_urdf>
   <!-- end effector -->

File: reach_description/description/alpha_5/urdf.xacro (robot description, xacro)
@@ -2,6 +2,7 @@
 <robot xmlns:xacro="http://ros.org/wiki/xacro">
   <xacro:macro name="alpha_5_urdf"
-               params="parent prefix *origin">
+               params="parent prefix *origin mount_rotation:=^0">
     <!-- links -->
+    <!-- the distance from the mount center to the base_link is xyz="0.0374 0 0.0225" -->
     <link name="${prefix}base_link">
       <visual>
@@ -9,5 +10,5 @@
           <mesh filename="file://$(find reach_description)/meshes/alpha_5/RS1-1010.dae" />
         </geometry>
-        <origin rpy="0 0 0"
+        <origin rpy="${mount_rotation} 0 0"
                 xyz="0 0 0" />
       </visual>
@@ -239,5 +240,5 @@
       <parent link="${prefix}base_link" />
       <child link="${prefix}m3_inline_link" />
-      <origin xyz="0.1614 0.004 0.0225"
+      <origin xyz="0.124 0.004 0"
               rpy="0 0 0" />
     </joint>
