Commit message: Added description files

File: reach_description/description/alpha_5/ros2_control.xacro (robot description, xacro)
@@ -3,6 +3,8 @@
   <xacro:macro name="alpha_system"
                params="prefix serial_port initial_positions_file use_sim:=^|false use_fake_hardware:=^true">
+    <xacro:property name="initial_positions_file"
+                    default="$(arg initial_positions_file)" />
     <xacro:property name="initial_positions"
-                    value="${xacro.load_yaml('$(arg initial_positions_file)')['initial_positions']}" />
+                    value="${xacro.load_yaml(initial_positions_file)['initial_positions']}" />
     <ros2_control name="ReachAlpha5"
                   type="system">

Commit message: Added simulation support

File: reach_description/description/alpha_5/ros2_control.xacro (robot description, xacro)
@@ -1,6 +1,7 @@
 <?xml version="1.0"?>
 <robot xmlns:xacro="http://www.ros.org/wiki/xacro">
-  <xacro:macro name="alpha_system"
+  <xacro:macro name="alpha_5_system"
                params="prefix serial_port initial_positions_file use_sim:=^|false use_mock_hardware:=^true">
+    <!-- load the initial positions for simulation -->
     <xacro:property name="initial_positions_file"
                     default="$(arg initial_positions_file)" />
@@ -9,4 +10,5 @@
     <ros2_control name="ReachAlpha5"
                   type="system">
+      <!-- use the GazeboSimSystem for simulation -->
       <xacro:if value="$(arg use_sim)">
         <hardware>
@@ -14,4 +16,5 @@
         </hardware>
       </xacro:if>
+      <!-- use either the mock interface or real interface if not using simulation -->
       <xacro:unless value="$(arg use_sim)">
         <hardware>
@@ -25,4 +28,6 @@
         </hardware>
       </xacro:unless>
+      <!-- joints -->
+      <!-- we need to include the device ID parameter for ros2_control -->
       <joint name="${prefix}axis_a">
         <param name="device_id">1</param>
@@ -35,4 +40,5 @@
           <param name="max">0.003</param>
         </command_interface>
+        <command_interface name="effort" />
         <state_interface name="position">
           <param name="initial_value">${initial_positions['axis_a']}</param>
@@ -41,5 +47,7 @@
           <param name="initial_value">0.0</param>
         </state_interface>
-        <state_interface name="effort" />
+        <state_interface name="effort">
+          <param name="initial_value">0.0</param>
+        </state_interface>
       </joint>
       <joint name="${prefix}axis_b">
@@ -53,4 +61,5 @@
           <param name="max">0.8726646</param>
         </command_interface>
+        <command_interface name="effort" />
         <state_interface name="position">
           <param name="initial_value">${initial_positions['axis_b']}</param>
@@ -59,5 +68,7 @@
           <param name="initial_value">0.0</param>
         </state_interface>
-        <state_interface name="effort" />
+        <state_interface name="effort">
+          <param name="initial_value">0.0</param>
+        </state_interface>
       </joint>
       <joint name="${prefix}axis_c">
@@ -71,4 +82,5 @@
           <param name="max">0.5235988</param>
         </command_interface>
+        <command_interface name="effort" />
         <state_interface name="position">
           <param name="initial_value">${initial_positions['axis_c']}</param>
@@ -77,5 +89,7 @@
           <param name="initial_value">0.0</param>
         </state_interface>
-        <state_interface name="effort" />
+        <state_interface name="effort">
+          <param name="initial_value">0.0</param>
+        </state_interface>
       </joint>
       <joint name="${prefix}axis_d">
@@ -89,4 +103,5 @@
           <param name="max">0.5235988</param>
         </command_interface>
+        <command_interface name="effort" />
         <state_interface name="position">
           <param name="initial_value">${initial_positions['axis_d']}</param>
@@ -95,5 +110,7 @@
           <param name="initial_value">0.0</param>
         </state_interface>
-        <state_interface name="effort" />
+        <state_interface name="effort">
+          <param name="initial_value">0.0</param>
+        </state_interface>
       </joint>
       <joint name="${prefix}axis_e">
@@ -107,4 +124,5 @@
           <param name="max">0.5235988</param>
         </command_interface>
+        <command_interface name="effort" />
         <state_interface name="position">
           <param name="initial_value">${initial_positions['axis_e']}</param>
@@ -113,5 +131,7 @@
           <param name="initial_value">0.0</param>
         </state_interface>
-        <state_interface name="effort" />
+        <state_interface name="effort">
+          <param name="initial_value">0.0</param>
+        </state_interface>
       </joint>
     </ros2_control>

File: reach_description/description/alpha_5/standard_jaws.config.xacro (robot description, xacro)
@@ -6,4 +6,5 @@
   <xacro:include filename="$(find reach_description)/description/alpha_5/ros2_control.xacro" />
   <xacro:include filename="$(find reach_description)/description/alpha_5/end_effectors/standard_jaws.urdf.xacro" />
+  <xacro:include filename="$(find reach_description)/description/alpha_5/gz.xacro" />
   <!-- parameters -->
   <xacro:arg name="use_mock_hardware"
@@ -17,4 +18,6 @@
   <xacro:arg name="parent"
              default="world" />
+  <xacro:arg name="controllers_file"
+             default="$(find reach_description)/config/alpha_5/controllers.yaml" />
   <!-- initial positions used for simulation -->
   <xacro:arg name="initial_positions_file"
@@ -27,9 +30,9 @@
   <link name="world" />
   <!-- arm -->
-  <xacro:alpha_urdf parent="$(arg parent)"
-                    prefix="${prefix}">
+  <xacro:alpha_5_urdf parent="$(arg parent)"
+                      prefix="${prefix}">
     <origin xyz="0 0 0"
             rpy="0 0 0" />
-  </xacro:alpha_urdf>
+  </xacro:alpha_5_urdf>
   <!-- end effector -->
   <xacro:standard_jaws parent="${prefix}rs1_124_link"
@@ -38,8 +41,12 @@
   </xacro:standard_jaws>
   <!-- ros2_control interface -->
-  <xacro:alpha_system prefix="${prefix}"
-                      serial_port="$(arg serial_port)"
-                      initial_positions_file="$(arg initial_positions_file)"
-                      use_sim="${use_sim}"
-                      use_mock_hardware="$(arg use_mock_hardware)" />
+  <xacro:alpha_5_system prefix="${prefix}"
+                        serial_port="$(arg serial_port)"
+                        initial_positions_file="$(arg initial_positions_file)"
+                        use_sim="${use_sim}"
+                        use_mock_hardware="$(arg use_mock_hardware)" />
+  <xacro:if value="$(arg use_sim)">
+    <xacro:alpha_5_gazebo prefix="${prefix}"
+                          controllers_file="$(arg controllers_file)" />
+  </xacro:if>
 </robot>

File: reach_description/description/alpha_5/urdf.xacro (robot description, xacro)
@@ -1,5 +1,5 @@
 <?xml version="1.0"?>
 <robot xmlns:xacro="http://ros.org/wiki/xacro">
-  <xacro:macro name="alpha_urdf"
+  <xacro:macro name="alpha_5_urdf"
                params="parent prefix *origin">
     <!-- links -->

Commit message: Added joint limit configuration file

File: reach_description/description/alpha_5/ros2_control.xacro (robot description, xacro)
@@ -2,5 +2,5 @@
 <robot xmlns:xacro="http://www.ros.org/wiki/xacro">
   <xacro:macro name="alpha_5_system"
-               params="prefix serial_port initial_positions_file use_sim:=^|false use_mock_hardware:=^true">
+               params="prefix serial_port initial_positions_file joint_limits_file use_sim:=^|false use_mock_hardware:=^true">
     <!-- load the initial positions for simulation -->
     <xacro:property name="initial_positions_file"
@@ -8,4 +8,9 @@
     <xacro:property name="initial_positions"
                     value="${xacro.load_yaml(initial_positions_file)['initial_positions']}" />
+    <!-- load the joint limits -->
+    <xacro:property name="joint_limits_file"
+                    default="$(arg joint_limits_file)" />
+    <xacro:property name="joint_limits"
+                    value="${xacro.load_yaml(joint_limits_file)['joint_limits']}" />
     <ros2_control name="ReachAlpha5"
                   type="system">
@@ -33,6 +38,6 @@
         <param name="device_id">1</param>
         <command_interface name="position">
-          <param name="min">0</param>
-          <param name="max">0.015</param>
+          <param name="min">${joint_limits['axis_a']['min_position']}</param>
+          <param name="max">${joint_limits['axis_a']['max_position']}</param>
         </command_interface>
         <command_interface name="velocity">
@@ -54,6 +59,6 @@
         <param name="device_id">2</param>
         <command_interface name="position">
-          <param name="min">0</param>
-          <param name="max">3.22</param>
+          <param name="min">${joint_limits['axis_b']['min_position']}</param>
+          <param name="max">${joint_limits['axis_b']['max_position']}</param>
         </command_interface>
         <command_interface name="velocity">
@@ -75,6 +80,6 @@
         <param name="device_id">3</param>
         <command_interface name="position">
-          <param name="min">0</param>
-          <param name="max">3.22</param>
+          <param name="min">${joint_limits['axis_c']['min_position']}</param>
+          <param name="max">${joint_limits['axis_c']['max_position']}</param>
         </command_interface>
         <command_interface name="velocity">
@@ -96,6 +101,6 @@
         <param name="device_id">4</param>
         <command_interface name="position">
-          <param name="min">0</param>
-          <param name="max">3.49</param>
+          <param name="min">${joint_limits['axis_d']['min_position']}</param>
+          <param name="max">${joint_limits['axis_d']['max_position']}</param>
         </command_interface>
         <command_interface name="velocity">
@@ -117,6 +122,6 @@
         <param name="device_id">5</param>
         <command_interface name="position">
-          <param name="min">0</param>
-          <param name="max">6.14</param>
+          <param name="min">${joint_limits['axis_e']['min_position']}</param>
+          <param name="max">${joint_limits['axis_e']['max_position']}</param>
         </command_interface>
         <command_interface name="velocity">

File: reach_description/description/alpha_5/standard_jaws/alpha_5.config.xacro (robot description, xacro)
@@ -20,4 +20,6 @@
   <xacro:arg name="controllers_file"
              default="$(find reach_description)/config/alpha_5/controllers.yaml" />
+  <xacro:arg name="joint_limits_file"
+             default="$(find reach_description)/config/alpha_5/joint_limits.yaml" />
   <xacro:arg name="mount_rotation"
              default="0" />
@@ -33,5 +35,6 @@
   <!-- arm -->
   <xacro:alpha_5_urdf parent="$(arg parent)"
-                      prefix="${prefix}">
+                      prefix="${prefix}"
+                      joint_limits_file="$(arg joint_limits_file)">
     <origin xyz="0.0374 0 0.0225"
             rpy="$(arg mount_rotation) 0 0" />
@@ -46,4 +49,5 @@
                         serial_port="$(arg serial_port)"
                         initial_positions_file="$(arg initial_positions_file)"
+                        joint_limits_file="$(arg joint_limits_file)"
                         use_sim="${use_sim}"
                         use_mock_hardware="$(arg use_mock_hardware)" />

File: reach_description/description/alpha_5/urdf.xacro (robot description, xacro)
@@ -2,5 +2,11 @@
 <robot xmlns:xacro="http://ros.org/wiki/xacro">
   <xacro:macro name="alpha_5_urdf"
-               params="parent prefix *origin mount_rotation:=^0">
+               params="parent prefix *origin joint_limits_file mount_rotation:=^0">
+    <!-- dynamically load the joint limits from a configuration file -->
+    <!-- this lets us modify a configuration file instead of requiring the implementation of a new URDF -->
+    <xacro:property name="joint_limits_file"
+                    default="$(arg joint_limits_file)" />
+    <xacro:property name="joint_limits"
+                    value="${xacro.load_yaml(joint_limits_file)['joint_limits']}" />
     <!-- links -->
     <!-- the distance from the mount center to the base_link is xyz="0.0374 0 0.0225" -->
@@ -250,6 +256,6 @@
       <axis xyz="0 0 1" />
       <limit effort="9.0"
-             lower="0.0"
-             upper="6.10"
+             lower="${joint_limits['axis_e']['min_position']}"
+             upper="${joint_limits['axis_e']['max_position']}"
              velocity="0.5" />
     </joint>
@@ -261,6 +267,6 @@
       <axis xyz="0 1 0" />
       <limit effort="9.0"
-             lower="-3.49"
-             upper="3.49"
+             lower="${joint_limits['axis_d']['min_position']}"
+             upper="${joint_limits['axis_d']['max_position']}"
              velocity="0.5" />
     </joint>
@@ -273,6 +279,6 @@
       <axis xyz="0 1 0" />
       <limit effort="9.0"
-             lower="0.0"
-             upper="3.22"
+             lower="${joint_limits['axis_c']['min_position']}"
+             upper="${joint_limits['axis_c']['max_position']}"
              velocity="0.5" />
     </joint>
@@ -285,6 +291,6 @@
       <axis xyz="0 0 -1" />
       <limit effort="9.0"
-             lower="0.0"
-             upper="3.22"
+             lower="${joint_limits['axis_b']['min_position']}"
+             upper="${joint_limits['axis_b']['max_position']}"
              velocity="0.5" />
     </joint>
@@ -304,6 +310,6 @@
       <axis xyz="0 0 1" />
       <limit effort="10"
-             lower="0"
-             upper="0.015"
+             lower="${joint_limits['axis_a']['min_position']}"
+             upper="${joint_limits['axis_a']['max_position']}"
              velocity="10" />
     </joint>
